File: ui-tile-1/ui-tile-kicad/lcd.kicad_sch (KiCad schematic)
At the start: 1 part

Commit message: finished schematic electricals
Parts:
- added Q1: 2N7002, jlcpcb:SOT-23-3_L2.9-W1.3-P1.90-LS2.4-BR, symbol jlcpcb:2N7002
- added R10: 100, jlcpcb:R0402, symbol jlcpcb:0402WGF1000TCE
- added R11: 68, jlcpcb:R0603, symbol jlcpcb:0603WAF680JT5E
- added R12: 10k, jlcpcb:R0402, symbol jlcpcb:0402WGF1002TCE
Connections:
- net GND: now reaches LCD1.1 (GND)
- net GND: now also LCD1.12 (GND), Q1.2 (S), R12.1
- net +3V3: now reaches LCD1.10 (FCS)
- net +3V3: now also LCD1.11 (VCC), LCD1.14 (FCS), LCD1.2 (VCC)
- net at LCD1.13 (BLA): now also R11.1
- net SCK: now reaches LCD1.16 (CLK)
- net SCK: now also LCD1.3 (CLK)
- net MOSI: now reaches LCD1.17 (SDA)
- net MOSI: now also LCD1.4 (SDA)
- net DC: now reaches LCD1.18 (DC)
- net DC: now also LCD1.6 (DC)
- net RES: now reaches LCD1.19 (RES)
- net RES: now also LCD1.5 (RES)
- net CS: now reaches LCD1.20 (CS1)
- net CS: now also LCD1.7 (CS1)
- net at LCD1.8 (BLK): now also Q1.3 (D)
- new net: Q1.1 (G), R10.2, R12.2
- new net BL: R10.1
- new net VSYS: R11.2
- no-connect marks 0 -> 2
Other:
- moved on the sheet: LCD1
