File: ui-tile-1/ui-tile-kicad/ui-tile-kicad.kicad_pcb (KiCad board)
At the start: 2 copper layers, 46 parts, among them SW1 SKRPABE010, SW2 SKRPABE010, SW3 EC11E15244G1, SW4 EC11E15244G1, SW5 EC11E15244G1, SW6 EC11E15244G1, U1 RP2040, U2 W25Q16JVUXIQ, U3 NCP1117ST33T3G, X1 12MHz

Commit message: finished schematic electricals
Parts:
- added H1: PZ254V-11-08P, jlcpcb:HDR-TH_8P-P2.54-V-M, B.Cu at (176.0, 94.2)
- added H2: PZ254V-11-08P, jlcpcb:HDR-TH_8P-P2.54-V-M, B.Cu at (87.5, 95.0)
- added Q1: 2N7002, jlcpcb:SOT-23-3_L2.9-W1.3-P1.90-LS2.4-BR, F.Cu at (143.2, 132.4)
- added R10: 100, jlcpcb:R0402, F.Cu at (139.7, 131.3)
- added R11: 68, jlcpcb:R0603, F.Cu at (143.2, 135.7)
- added R12: 10k, jlcpcb:R0402, F.Cu at (139.7, 133.5)
- added U4: 74AHCT1G125W5-7, jlcpcb:SOT-25-5_L3.0-W1.6-P0.95-LS2.8-BL, B.Cu at (147.2, 128.8)
- moved LED5 66.0 mm to (169.8, 68.5)
- moved LED3 64.5 mm to (97.2, 67.0)
- moved LED4 64.3 mm to (97.2, 121.0)
- moved LED6 61.8 mm to (165.5, 124.8)
- moved SW5 28.5 mm to (161.2, 80.8)
- moved SW6 24.8 mm to (162.0, 110.0)
- moved SW4 4.37 mm to (103.0, 108.0)
Connections:
- C13 pad 2: /rp2040/VSYS -> VSYS
- C14 pad 2: /rp2040/VSYS -> VSYS
- D1 pad 1: /rp2040/VSYS -> VSYS
- D2 pad 1: /rp2040/VSYS -> VSYS
- D2 pad 2: /rp2040/+5V -> +5V
- LCD1 pad 1: unconnected-(LCD1-GND-Pad1) -> GND
- LCD1 pad 10: unconnected-(LCD1-FCS-Pad10) -> +3V3
- LCD1 pad 11: unconnected-(LCD1-VCC-Pad11) -> +3V3
- LCD1 pad 12: unconnected-(LCD1-GND-Pad12) -> GND
- LCD1 pad 13: unconnected-(LCD1-BLA-Pad13) -> Net-(LCD1-BLA)
- LCD1 pad 14: unconnected-(LCD1-FCS-Pad14) -> +3V3
- LCD1 pad 16: unconnected-(LCD1-CLK-Pad16) -> /lcd/SCK
- LCD1 pad 17: unconnected-(LCD1-SDA-Pad17) -> /lcd/MOSI
- LCD1 pad 18: unconnected-(LCD1-DC-Pad18) -> /lcd/DC
- LCD1 pad 19: unconnected-(LCD1-RES-Pad19) -> /lcd/RES
- LCD1 pad 2: unconnected-(LCD1-VCC-Pad2) -> +3V3
- LCD1 pad 20: unconnected-(LCD1-CS1-Pad20) -> /lcd/CS
- LCD1 pad 3: unconnected-(LCD1-CLK-Pad3) -> /lcd/SCK
- LCD1 pad 4: unconnected-(LCD1-SDA-Pad4) -> /lcd/MOSI
- LCD1 pad 5: unconnected-(LCD1-RES-Pad5) -> /lcd/RES
- LCD1 pad 6: unconnected-(LCD1-DC-Pad6) -> /lcd/DC
- LCD1 pad 7: unconnected-(LCD1-CS1-Pad7) -> /lcd/CS
- LCD1 pad 8: unconnected-(LCD1-BLK-Pad8) -> Net-(LCD1-BLK)
- LED3 pad 1: unconnected-(LED3-VDD-Pad1) -> VSYS
- LED3 pad 2: unconnected-(LED3-DOUT-Pad2) -> Net-(LED3-DOUT)
- LED3 pad 3: unconnected-(LED3-VSS-Pad3) -> GND
- LED3 pad 4: unconnected-(LED3-DIN-Pad4) -> /leds/LED
- LED4 pad 1: unconnected-(LED4-VDD-Pad1) -> VSYS
- LED4 pad 2: unconnected-(LED4-DOUT-Pad2) -> Net-(LED4-DOUT)
- LED4 pad 3: unconnected-(LED4-VSS-Pad3) -> GND
- LED4 pad 4: unconnected-(LED4-DIN-Pad4) -> Net-(LED3-DOUT)
- LED5 pad 1: unconnected-(LED5-VDD-Pad1) -> VSYS
- LED5 pad 2: unconnected-(LED5-DOUT-Pad2) -> Net-(LED5-DOUT)
- LED5 pad 3: unconnected-(LED5-VSS-Pad3) -> GND
- LED5 pad 4: unconnected-(LED5-DIN-Pad4) -> Net-(LED4-DOUT)
- LED6 pad 1: unconnected-(LED6-VDD-Pad1) -> VSYS
- LED6 pad 3: unconnected-(LED6-VSS-Pad3) -> GND
- LED6 pad 4: unconnected-(LED6-DIN-Pad4) -> Net-(LED5-DOUT)
- R9 pad 1: /rp2040/VSYS -> VSYS
- SW3 pad 6: unconnected-(SW3-Pad6) -> GND
- SW3 pad 7: unconnected-(SW3-Pad7) -> GND
- SW3 pad A: unconnected-(SW3-PadA) -> /encoders/Enc1_A
- SW3 pad B: unconnected-(SW3-PadB) -> /encoders/Enc1_B
- SW3 pad C: unconnected-(SW3-PadC) -> GND
- SW3 pad D: unconnected-(SW3-PadD) -> /encoders/Enc1_SW
- SW3 pad E: unconnected-(SW3-PadE) -> GND
- SW4 pad 6: unconnected-(SW4-Pad6) -> GND
- SW4 pad 7: unconnected-(SW4-Pad7) -> GND
- SW4 pad A: unconnected-(SW4-PadA) -> /encoders/Enc2_A
- SW4 pad B: unconnected-(SW4-PadB) -> /encoders/Enc2_B
- SW4 pad C: unconnected-(SW4-PadC) -> GND
- SW4 pad D: unconnected-(SW4-PadD) -> /encoders/Enc2_SW
- SW4 pad E: unconnected-(SW4-PadE) -> GND
- SW5 pad 6: unconnected-(SW5-Pad6) -> GND
- SW5 pad 7: unconnected-(SW5-Pad7) -> GND
- SW5 pad A: unconnected-(SW5-PadA) -> /encoders/Enc3_A
- SW5 pad B: unconnected-(SW5-PadB) -> /encoders/Enc3_B
- SW5 pad C: unconnected-(SW5-PadC) -> GND
- SW5 pad D: unconnected-(SW5-PadD) -> /encoders/Enc3_SW
- SW5 pad E: unconnected-(SW5-PadE) -> GND
- SW6 pad 6: unconnected-(SW6-Pad6) -> GND
- SW6 pad 7: unconnected-(SW6-Pad7) -> GND
- SW6 pad A: unconnected-(SW6-PadA) -> /encoders/Enc4_A
- SW6 pad B: unconnected-(SW6-PadB) -> /encoders/Enc4_B
- SW6 pad C: unconnected-(SW6-PadC) -> GND
- SW6 pad D: unconnected-(SW6-PadD) -> /encoders/Enc4_SW
- SW6 pad E: unconnected-(SW6-PadE) -> GND
- U1 pad 11: unconnected-(U1-GPIO8-Pad11) -> /lcd/DC
- U1 pad 12: unconnected-(U1-GPIO9-Pad12) -> /lcd/CS
- U1 pad 13: unconnected-(U1-GPIO10-Pad13) -> /lcd/SCK
- U1 pad 14: unconnected-(U1-GPIO11-Pad14) -> /lcd/MOSI
- U1 pad 2: unconnected-(U1-GPIO0-Pad2) -> /headers/MISO
- U1 pad 27: unconnected-(U1-GPIO16-Pad27) -> /encoders/Enc1_A
- U1 pad 28: unconnected-(U1-GPIO17-Pad28) -> /encoders/Enc1_B
- U1 pad 29: unconnected-(U1-GPIO18-Pad29) -> /encoders/Enc1_SW
- U1 pad 3: unconnected-(U1-GPIO1-Pad3) -> /headers/CS
- U1 pad 30: unconnected-(U1-GPIO19-Pad30) -> /encoders/Enc2_A
- U1 pad 31: unconnected-(U1-GPIO20-Pad31) -> /encoders/Enc2_B
- U1 pad 32: unconnected-(U1-GPIO21-Pad32) -> /encoders/Enc2_SW
- U1 pad 34: unconnected-(U1-GPIO22-Pad34) -> /encoders/Enc3_A
- U1 pad 35: unconnected-(U1-GPIO23-Pad35) -> /encoders/Enc3_B
- U1 pad 36: unconnected-(U1-GPIO24-Pad36) -> /encoders/Enc3_SW
- U1 pad 37: unconnected-(U1-GPIO25-Pad37) -> /encoders/Enc4_A
- U1 pad 38: unconnected-(U1-GPIO26_ADC0-Pad38) -> /encoders/Enc4_B
- U1 pad 39: unconnected-(U1-GPIO27_ADC1-Pad39) -> /encoders/Enc4_SW
- U1 pad 4: unconnected-(U1-GPIO2-Pad4) -> /headers/SCK
- U1 pad 5: unconnected-(U1-GPIO3-Pad5) -> /headers/MOSI
- U1 pad 6: unconnected-(U1-GPIO4-Pad6) -> /headers/IRQ
- U1 pad 7: unconnected-(U1-GPIO5-Pad7) -> /leds/LED_3V3
- U1 pad 8: unconnected-(U1-GPIO6-Pad8) -> /lcd/RES
- U1 pad 9: unconnected-(U1-GPIO7-Pad9) -> /lcd/BL
- U3 pad 3: /rp2040/VSYS -> VSYS

Commit message: preparing for pcb layout
Parts:
- added C18: 100nF, jlcpcb:C0402, F.Cu at (90.4, 67.0)
- added C19: 100nF, jlcpcb:C0402, F.Cu at (163.8, 67.8)
- added C20: 100nF, jlcpcb:C0402, F.Cu at (91.6, 120.6)
- added C21: 100nF, jlcpcb:C0402, F.Cu at (170.4, 124.4)
- added C22: 10uF, jlcpcb:C0805, F.Cu at (100.2, 59.0)
- added R13: 470, jlcpcb:R0402, F.Cu at (103.6, 62.6)
- moved USBC1 141.8 mm to (142.2, 165.5), turned to 0 degrees
- moved LED1 141.5 mm to (125.9, 164.5), turned to 90 degrees
- moved C13 141.0 mm to (129.2, 164.7), turned to 180 degrees
- moved C14 137.5 mm to (129.2, 163.0), turned to 180 degrees
- moved R9 135.1 mm to (125.9, 161.2), turned to -90 degrees
- moved U3 128.1 mm to (131.4, 158.5), turned to 180 degrees
- moved R4 127.5 mm to (144.7, 158.1), turned to 0 degrees
- moved R3 127.0 mm to (141.9, 158.1), turned to 0 degrees
- moved D1 124.2 mm to (120.8, 154.5), turned to 180 degrees
- moved C1 120.3 mm to (148.2, 154.0), turned to 90 degrees
- moved LED2 120.0 mm to (136.4, 154.7), turned to 90 degrees
- moved C5 119.9 mm to (146.9, 154.0), turned to 90 degrees
- moved R1 119.5 mm to (145.7, 154.0), turned to -90 degrees
- moved R2 119.2 mm to (144.4, 154.0), turned to -90 degrees
- moved U2 119.2 mm to (151.4, 152.7), turned to -90 degrees
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Connections:
- U4 pad 4: /leds/LED -> Net-(U4-Y)

Commit message: progress on pcb layout
Parts:
- U4: moved to F.Cu
- moved H1 57.6 mm to (131.0, 130.2), turned to 180 degrees
- moved H2 55.1 mm to (131.6, 62.0), turned to 180 degrees
- moved R9 50.1 mm to (174.8, 150.2), turned to 180 degrees
- moved LED1 47.3 mm to (171.7, 152.6), turned to 0 degrees
- moved C11 46.5 mm to (110.7, 120.0), turned to 0 degrees
- moved C12 43.4 mm to (107.8, 121.8)
- moved X1 43.1 mm to (110.5, 122.3)
- moved R5 43.0 mm to (109.0, 124.6)
- moved C1 42.9 mm to (108.8, 137.0)
- moved C5 42.8 mm to (107.6, 137.0)
- moved R1 42.8 mm to (106.4, 137.0), turned to 90 degrees
- moved C2 42.7 mm to (106.4, 123.8)
- moved C8 42.7 mm to (107.4, 123.8)
- moved R2 42.7 mm to (105.2, 137.0), turned to 90 degrees
- moved C3 41.7 mm to (104.6, 135.7), turned to 45 degrees
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Connections:
- net Net-(U1-USB_DM) renamed /rp2040/USB_DN
- net Net-(U1-USB_DP) renamed /rp2040/USB_DP
- U1 pad 11: /lcd/DC -> /lcd/MOSI
- U1 pad 12: /lcd/CS -> /lcd/DC
- U1 pad 13: /lcd/SCK -> /lcd/RES
- U1 pad 14: /lcd/MOSI -> /lcd/CS
- U1 pad 27: /encoders/Enc1_A -> /encoders/Enc4_B
- U1 pad 28: /encoders/Enc1_B -> /encoders/Enc4_A
- U1 pad 29: /encoders/Enc1_SW -> /encoders/Enc4_SW
- U1 pad 30: /encoders/Enc2_A -> /encoders/Enc3_B
- U1 pad 31: /encoders/Enc2_B -> /encoders/Enc3_A
- U1 pad 32: /encoders/Enc2_SW -> /encoders/Enc3_SW
- U1 pad 34: /encoders/Enc3_A -> /encoders/Enc1_B
- U1 pad 35: /encoders/Enc3_B -> /encoders/Enc1_A
- U1 pad 36: /encoders/Enc3_SW -> /encoders/Enc1_SW
- U1 pad 37: /encoders/Enc4_A -> /encoders/Enc2_B
- U1 pad 38: /encoders/Enc4_B -> /encoders/Enc2_A
- U1 pad 39: /encoders/Enc4_SW -> /encoders/Enc2_SW
- U1 pad 8: /lcd/RES -> /lcd/BL
- U1 pad 9: /lcd/BL -> /lcd/SCK
Routing:
- net /encoders/Enc3_SW: track 0.00 -> 88.3 mm
- net /encoders/Enc3_B: track 0.00 -> 76.4 mm
- net /encoders/Enc1_SW: track 0.00 -> 76.2 mm
- net /encoders/Enc3_A: track 0.00 -> 74.4 mm
- net /encoders/Enc4_B: track 0.00 -> 72.2 mm
- net /encoders/Enc4_A: track 0.00 -> 67.0 mm
- net /encoders/Enc4_SW: track 0.00 -> 66.7 mm
- net /encoders/Enc1_A: track 0.00 -> 59.9 mm
- net /encoders/Enc1_B: track 0.00 -> 55.0 mm
- net /encoders/Enc2_SW: track 0.00 -> 52.1 mm
- net /encoders/Enc2_A: track 0.00 -> 40.2 mm, vias 0 -> 2
- net /encoders/Enc2_B: track 0.00 -> 36.5 mm, vias 0 -> 3
- net GND: track 0.00 -> 31.1 mm, vias 0 -> 23
- net /rp2040/USB_D-: track 2.92 -> 27.1 mm, vias 0 -> 2
- net /lcd/SCK: track 0.00 -> 22.6 mm
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- added copper zone on F.Cu, net +3V3
- added copper zone on In1.Cu, net GND
Other:
- copper layers 2 -> 4
