File: ui-tile-1/ui-tile-kicad/rp2040.kicad_sch (KiCad schematic)
At the start: 37 parts, among them SW1 SKRPABE010, SW2 SKRPABE010, U1 RP2040, U2 W25Q16JVUXIQ, U3 NCP1117ST33T3G, X1 12MHz

Commit message: finished schematic electricals
Connections:
- net LCD_DC: now reaches U1.11 (GPIO8)
- net LCD_CS: now reaches U1.12 (GPIO9)
- net LCD_SCK: now reaches U1.13 (GPIO10)
- net LCD_MOSI: now reaches U1.14 (GPIO11)
- net MB_MISO: now reaches U1.2 (GPIO0)
- net Enc1_A: now reaches U1.27 (GPIO16)
- net Enc1_B: now reaches U1.28 (GPIO17)
- net Enc1_SW: now reaches U1.29 (GPIO18)
- net MB_CS: now reaches U1.3 (GPIO1)
- net Enc2_A: now reaches U1.30 (GPIO19)
- net Enc2_B: now reaches U1.31 (GPIO20)
- net Enc2_SW: now reaches U1.32 (GPIO21)
- net Enc3_A: now reaches U1.34 (GPIO22)
- net Enc3_B: now reaches U1.35 (GPIO23)
- net Enc3_SW: now reaches U1.36 (GPIO24)
- net Enc4_A: now reaches U1.37 (GPIO25)
- net Enc4_B: now reaches U1.38 (GPIO26_ADC0)
- net Enc4_SW: now reaches U1.39 (GPIO27_ADC1)
- net MB_SCK: now reaches U1.4 (GPIO2)
- net MB_MOSI: now reaches U1.5 (GPIO3)
- net MB_IRQ: now reaches U1.6 (GPIO4)
- net LED_OUT: now reaches U1.7 (GPIO5)
- net LCD_RST: now reaches U1.8 (GPIO6)
- net LCD_BL: now reaches U1.9 (GPIO7)
- no-connect marks 38 -> 14

Commit message: progress on pcb layout
Connections:
- net Enc1_A: now also U1.35 (GPIO23); no longer U1.27 (GPIO16)
- net Enc1_B: now also U1.34 (GPIO22); no longer U1.28 (GPIO17)
- net Enc1_SW: now also U1.36 (GPIO24); no longer U1.29 (GPIO18)
- net Enc2_A: now also U1.38 (GPIO26_ADC0); no longer U1.30 (GPIO19)
- net Enc2_B: now also U1.37 (GPIO25); no longer U1.31 (GPIO20)
- net Enc2_SW: now also U1.39 (GPIO27_ADC1); no longer U1.32 (GPIO21)
- net Enc3_A: now also U1.31 (GPIO20); no longer U1.34 (GPIO22)
- net Enc3_B: now also U1.30 (GPIO19); no longer U1.35 (GPIO23)
- net Enc3_SW: now also U1.32 (GPIO21); no longer U1.36 (GPIO24)
- net Enc4_A: now also U1.28 (GPIO17); no longer U1.37 (GPIO25)
- net Enc4_B: now also U1.27 (GPIO16); no longer U1.38 (GPIO26_ADC0)
- net Enc4_SW: now also U1.29 (GPIO18); no longer U1.39 (GPIO27_ADC1)
- net LCD_BL: now also U1.8 (GPIO6); no longer U1.9 (GPIO7)
- net LCD_CS: now also U1.14 (GPIO11); no longer U1.12 (GPIO9)
- net LCD_DC: now also U1.12 (GPIO9); no longer U1.11 (GPIO8)
- net LCD_MOSI: now also U1.11 (GPIO8); no longer U1.14 (GPIO11)
- net LCD_RST: now also U1.13 (GPIO10); no longer U1.8 (GPIO6)
- net LCD_SCK: now also U1.9 (GPIO7); no longer U1.13 (GPIO10)
- net USB_DN: now reaches R2.2, U1.46 (USB_DM)
- net USB_DP: now reaches R1.2, U1.47 (USB_DP)
Changed lines of the file:
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@@
+	)
+	(junction
+		(at 106.68 71.12)
+		(diameter 0)
+		(color 0 0 0 0)
 	)
 	(junction
@@
 	)
 	(junction
+		(at 106.68 77.47)
+		(diameter 0)
+		(color 0 0 0 0)
+	)
+	(junction
 		(at 242.57 127)
 		(diameter 0)
@@
 	(wire
 		(pts
-			(xy 102.87 77.47) (xy 110.49 77.47)
+			(xy 102.87 77.47) (xy 106.68 77.47)
 		)
 		(stroke
@@
 	(wire
 		(pts
+			(xy 106.68 77.47) (xy 106.68 82.55)
+		)
+		(stroke
+			(width 0)
+			(type default)
+		)
+	)
+	(wire
+		(pts
 			(xy 190.5 48.26) (xy 190.5 50.8)
 		)
@@
 	(wire
 		(pts
+			(xy 106.68 66.04) (xy 119.38 66.04)
+		)
+		(stroke
+			(width 0)
+			(type default)
+		)
+	)
+	(wire
+		(pts
 			(xy 228.6 138.43) (xy 228.6 146.05)
 		)
@@
 	(wire
 		(pts
+			(xy 106.68 82.55) (xy 119.38 82.55)
+		)
+		(stroke
+			(width 0)
+			(type default)
+		)
+	)
+	(wire
+		(pts
 			(xy 102.87 90.17) (xy 128.27 90.17)
 		)
@@
 	(wire
 		(pts
+			(xy 106.68 77.47) (xy 110.49 77.47)
+		)
+		(stroke
+			(width 0)
+			(type default)
+		)
+	)
+	(wire
+		(pts
 			(xy 170.18 105.41) (xy 172.72 105.41)
 		)
@@
 		(pts
 			(xy 190.5 140.97) (xy 201.93 140.97)
+		)
+		(stroke
+			(width 0)
+			(type default)
+		)
+	)
+	(wire
+		(pts
+			(xy 106.68 71.12) (xy 106.68 66.04)
 		)
 		(stroke
@@
 		)
 	)
+	(label "USB_DP"
+		(at 119.38 66.04 0)
+		(effects
+			(font
+				(size 1.27 1.27)
+			)
+			(justify left bottom)
+		)
+	)
 	(label "+1V1"
 		(at 130.81 184.15 0)
@@
 		)
 	)
+	(label "USB_DN"
+		(at 119.38 82.55 0)
+		(effects
+			(font
+				(size 1.27 1.27)
+			)
+			(justify left bottom)
+		)
+	)
 	(label "XOUT"
 		(at 227.33 31.75 180)
@@
 		)
 	)
+	(hierarchical_label "LCD_CS"
+		(shape input)
+		(at 128.27 113.03 0)
+		(effects
+			(font
+				(size 1.27 1.27)
+			)
+			(justify left)
+		)
+	)
+	(hierarchical_label "Enc1_SW"
+		(shape input)
+		(at 128.27 146.05 0)
+		(effects
+			(font
+				(size 1.27 1.27)
+			)
+			(justify left)
+		)
+	)
+	(hierarchical_label "Enc2_B"
+		(shape input)
+		(at 128.27 148.59 0)
+		(effects
+			(font
+				(size 1.27 1.27)
+			)
+			(justify left)
+		)
+	)
 	(hierarchical_label "LCD_MOSI"
 		(shape input)
-		(at 128.27 113.03 0)
+		(at 128.27 105.41 0)
+		(effects
+			(font
+				(size 1.27 1.27)
+			)
+			(justify left)
+		)
+	)
+	(hierarchical_label "Enc1_A"
+		(shape input)
+		(at 128.27 143.51 0)
 		(effects
 			(font
@@
 	(hierarchical_label "Enc3_SW"
 		(shape input)
-		(at 128.27 146.05 0)
+		(at 128.27 138.43 0)
 		(effects
 			(font
@@
 		)
 	)
-	(hierarchical_label "Enc4_A"
+	(hierarchical_label "LCD_RST"
 		(shape input)
-		(at 128.27 148.59 0)
+		(at 128.27 110.49 0)
+		(effects
+			(font
+				(size 1.27 1.27)
+			)
+			(justify left)
+		)
+	)
+	(hierarchical_label "Enc4_SW"
+		(shape input)
+		(at 128.27 130.81 0)
+		(effects
+			(font
+				(size 1.27 1.27)
+			)
+			(justify left)
+		)
+	)
+	(hierarchical_label "Enc2_SW"
+		(shape input)
+		(at 128.27 156.21 0)
 		(effects
 			(font
@@
 	(hierarchical_label "LCD_DC"
 		(shape input)
-		(at 128.27 105.41 0)
+		(at 128.27 107.95 0)
 		(effects
 			(font
@@
 		)
 	)
-	(hierarchical_label "Enc3_B"
+	(hierarchical_label "Enc1_B"
 		(shape input)
-		(at 128.27 143.51 0)
+		(at 128.27 140.97 0)
 		(effects
 			(font
@@
 		)
 	)
-	(hierarchical_label "Enc2_SW"
+	(hierarchical_label "LCD_BL"
 		(shape input)
-		(at 128.27 138.43 0)
+		(at 128.27 100.33 0)
 		(effects
 			(font
@@
 	(hierarchical_label "LCD_SCK"
 		(shape input)
-		(at 128.27 110.49 0)
+		(at 128.27 102.87 0)
 		(effects
 			(font
@@
 		)
 	)
-	(hierarchical_label "Enc1_SW"
-		(shape input)
-		(at 128.27 130.81 0)
-		(effects
-			(font
-				(size 1.27 1.27)
-			)
-			(justify left)
-		)
-	)
-	(hierarchical_label "Enc4_SW"
-		(shape input)
-		(at 128.27 156.21 0)
-		(effects
-			(font
-				(size 1.27 1.27)
-			)
-			(justify left)
-		)
-	)
-	(hierarchical_label "LCD_CS"
-		(shape input)
-		(at 128.27 107.95 0)
-		(effects
-			(font
-				(size 1.27 1.27)
-			)
-			(justify left)
-		)
-	)
-	(hierarchical_label "Enc3_A"
-		(shape input)
-		(at 128.27 140.97 0)
-		(effects
-			(font
-				(size 1.27 1.27)
-			)
-			(justify left)
-		)
-	)
-	(hierarchical_label "LCD_RST"
-		(shape input)
-		(at 128.27 100.33 0)
-		(effects
-			(font
-				(size 1.27 1.27)
-			)
-			(justify left)
-		)
-	)
-	(hierarchical_label "LCD_BL"
-		(shape input)
-		(at 128.27 102.87 0)
-		(effects
-			(font
-				(size 1.27 1.27)
-			)
-			(justify left)
-		)
-	)
-	(hierarchical_label "Enc4_B"
+	(hierarchical_label "Enc2_A"
 		(shape input)
 		(at 128.27 153.67 0)
@@
 		)
 	)
-	(hierarchical_label "Enc2_B"
+	(hierarchical_label "Enc3_A"
 		(shape input)
 		(at 128.27 135.89 0)
@@
 		)
 	)
-	(hierarchical_label "Enc1_A"
+	(hierarchical_label "Enc4_B"
 		(shape input)
 		(at 128.27 125.73 0)
@@
 		)
 	)
-	(hierarchical_label "Enc2_A"
+	(hierarchical_label "Enc3_B"
 		(shape input)
 		(at 128.27 133.35 0)
@@
 		)
 	)
-	(hierarchical_label "Enc1_B"
+	(hierarchical_label "Enc4_A"
 		(shape input)
 		(at 128.27 128.27 0)

Commit message: finished first pass of pcb layout
Connections:
- net MB_CS: now also U1.2 (GPIO0); no longer U1.3 (GPIO1)
- net MB_MISO: now also U1.4 (GPIO2); no longer U1.2 (GPIO0)
- net MB_SCK: now also U1.3 (GPIO1); no longer U1.4 (GPIO2)
Changed lines of the file:
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@@
 		)
 	)
-	(hierarchical_label "MB_CS"
+	(hierarchical_label "MB_SCK"
 		(shape input)
 		(at 128.27 87.63 0)
@@
 		)
 	)
-	(hierarchical_label "MB_MISO"
+	(hierarchical_label "MB_CS"
 		(shape input)
 		(at 128.27 85.09 0)
@@
 		)
 	)
-	(hierarchical_label "MB_SCK"
+	(hierarchical_label "MB_MISO"
 		(shape input)
 		(at 128.27 90.17 0)
